Commit message: Fix: Add tf_prefix into xacro

File: catkin_ws/src/jackal/jackal_description/urdf/jackal.urdf.xacro (robot description, xacro)
@@ -18,5 +18,5 @@
   <material name="black"><color rgba="0.15 0.15 0.15 1.0" /></material>
   <xacro:macro name="wheel" params="prefix *joint_pose">
-    <link name="${prefix}_wheel_link">
+    <link name="$(arg tf_prefix)/${prefix}_wheel_link">
       <visual>
         <origin xyz="0 0 0" rpy="${PI/2} 0 0"/>
@@ -50,7 +50,7 @@
       <fdir1 value="1 0 0"/>
     </gazebo>
-    <joint name="${prefix}_wheel" type="continuous">
-      <parent link="chassis_link"/>
-      <child link="${prefix}_wheel_link" />
+    <joint name="$(arg tf_prefix)/${prefix}_wheel" type="continuous">
+      <parent link="$(arg tf_prefix)/chassis_link"/>
+      <child link="$(arg tf_prefix)/${prefix}_wheel_link" />
       <xacro:insert_block name="joint_pose" />
       <axis xyz="0 1 0" />
@@ -60,5 +60,5 @@
     <transmission name="${prefix}_wheel_trans">
       <type>transmission_interface/SimpleTransmission</type>
-      <joint name="${prefix}_wheel">
+      <joint name="$(arg tf_prefix)/${prefix}_wheel">
         <hardwareInterface>hardware_interface/VelocityJointInterface</hardwareInterface>
       </joint>
@@ -80,11 +80,11 @@
     <origin xyz="${-wheelbase/2} ${-track/2} ${wheel_vertical_offset}" rpy="0 0 0" />
   </xacro:wheel>
-  <link name="base_link"> </link>
-  <joint name="base_link_joint" type="fixed">
+  <link name="$(arg tf_prefix)/base_link"> </link>
+  <joint name="$(arg tf_prefix)/base_link_joint" type="fixed">
     <origin xyz="0 0 0" rpy="0 0 0" />
-    <parent link="base_link"/>
-    <child link="chassis_link" />
-  </joint>
-  <link name="chassis_link">
+    <parent link="$(arg tf_prefix)/base_link"/>
+    <child link="$(arg tf_prefix)/chassis_link" />
+  </joint>
+  <link name="$(arg tf_prefix)/chassis_link">
     <visual>
       <origin xyz="0 0 ${footprint_vertical_offset}" rpy="${PI/2} 0 ${PI/2}"/>
@@ -112,5 +112,5 @@
   </link>
   <xacro:unless value="$(optenv JACKAL_FRONT_ACCESSORY_FENDER 0)">
-    <link name="front_fender_link">
+    <link name="$(arg tf_prefix)/front_fender_link">
       <visual>
         <geometry>
@@ -122,5 +122,5 @@
   </xacro:unless>
   <xacro:if value="$(optenv JACKAL_FRONT_ACCESSORY_FENDER 0)">
-    <link name="front_fender_link">
+    <link name="$(arg tf_prefix)/front_fender_link">
       <visual>
         <geometry>
@@ -130,18 +130,18 @@
       </visual>
     </link>
-    <link name="front_fender_accessory_link"/>
-    <joint name="front_fender_accessory_joint" type="fixed">
+    <link name="$(arg tf_prefix)/front_fender_accessory_link"/>
+    <joint name="$(arg tf_prefix)/front_fender_accessory_joint" type="fixed">
       <origin xyz="0.25629 0 0.07455" rpy="${PI} 0 0" />
-      <parent link="front_fender_link" />
-      <child link="front_fender_accessory_link" />
+      <parent link="$(arg tf_prefix)/front_fender_link" />
+      <child link="$(arg tf_prefix)/front_fender_accessory_link" />
     </joint>
   </xacro:if>
-  <joint name="front_fender_joint" type="fixed">
+  <joint name="$(arg tf_prefix)/front_fender_joint" type="fixed">
     <origin xyz="0 0 0" rpy="0 0 0"/>
-    <parent link="chassis_link" />
-    <child link="front_fender_link" />
+    <parent link="$(arg tf_prefix)/chassis_link" />
+    <child link="$(arg tf_prefix)/front_fender_link" />
   </joint>
   <xacro:unless value="$(optenv JACKAL_REAR_ACCESSORY_FENDER 0)">
-    <link name="rear_fender_link">
+    <link name="$(arg tf_prefix)/rear_fender_link">
       <visual>
         <geometry>
@@ -153,5 +153,5 @@
   </xacro:unless>
   <xacro:if value="$(optenv JACKAL_REAR_ACCESSORY_FENDER 0)">
-    <link name="rear_fender_link">
+    <link name="$(arg tf_prefix)/rear_fender_link">
       <visual>
         <geometry>
@@ -161,15 +161,15 @@
       </visual>
     </link>
-    <link name="rear_fender_accessory_link"/>
-    <joint name="rear_fender_accessory_joint" type="fixed">
+    <link name="$(arg tf_prefix)/rear_fender_accessory_link"/>
+    <joint name="$(arg tf_prefix)/rear_fender_accessory_joint" type="fixed">
       <origin xyz="0.25629 0 0.07455" rpy="${PI} 0 0" />
-      <parent link="rear_fender_link" />
-      <child link="rear_fender_accessory_link" />
+      <parent link="$(arg tf_prefix)/rear_fender_link" />
+      <child link="$(arg tf_prefix)/rear_fender_accessory_link" />
     </joint>
   </xacro:if>
-  <joint name="rear_fender_joint" type="fixed">
+  <joint name="$(arg tf_prefix)/rear_fender_joint" type="fixed">
     <origin xyz="0 0 0" rpy="0 0 ${PI}"/>
-    <parent link="chassis_link" />
-    <child link="rear_fender_link" />
+    <parent link="$(arg tf_prefix)/chassis_link" />
+    <child link="$(arg tf_prefix)/rear_fender_link" />
   </joint>
   <!-- TODO: Make this internal_imu_link or something, and use a mixed-in xacro
@@ -177,5 +177,5 @@
        always points to the "active" IMU. When an upgrade IMU is connected, the
        internal_imu_link should remain, but imu_link should point to the upgrade one. -->
-  <link name="imu_link">
+  <link name="$(arg tf_prefix)/imu_link">
     <inertial>
       <mass value="0.001"/>
@@ -184,10 +184,10 @@
     </inertial>
   </link>
-  <joint name="imu_joint" type="fixed">
-    <parent link="chassis_link" />
-    <child link="imu_link" />
+  <joint name="$(arg tf_prefix)/imu_joint" type="fixed">
+    <parent link="$(arg tf_prefix)/chassis_link" />
+    <child link="$(arg tf_prefix)/imu_link" />
   </joint>
   <!-- TODO: Same note as applies to imu_link -->
-  <link name="navsat_link">
+  <link name="$(arg tf_prefix)/navsat_link">
     <visual>
       <geometry>
@@ -198,25 +198,25 @@
     </visual>
   </link>
-  <joint name="navsat_joint" type="fixed">
-    <parent link="chassis_link" />
-    <child link="navsat_link" />
+  <joint name="$(arg tf_prefix)/navsat_joint" type="fixed">
+    <parent link="$(arg tf_prefix)/chassis_link" />
+    <child link="$(arg tf_prefix)/navsat_link" />
     <origin xyz="-0.180 0.126 0.1815" />
   </joint>
-  <link name="mid_mount"></link>
-  <joint name="mid_mount_joint" type="fixed">
-    <parent link="chassis_link" />
-    <child link="mid_mount" />
+  <link name="$(arg tf_prefix)/mid_mount"></link>
+  <joint name="$(arg tf_prefix)/mid_mount_joint" type="fixed">
+    <parent link="$(arg tf_prefix)/chassis_link" />
+    <child link="$(arg tf_prefix)/mid_mount" />
     <origin xyz="0 0 ${chassis_height}" />
   </joint>
-  <link name="rear_mount"></link>
-  <joint name="rear_mount_joint" type="fixed">
-    <parent link="mid_mount" />
-    <child link="rear_mount" />
+  <link name="$(arg tf_prefix)/rear_mount"></link>
+  <joint name="$(arg tf_prefix)/rear_mount_joint" type="fixed">
+    <parent link="$(arg tf_prefix)/mid_mount" />
+    <child link="$(arg tf_prefix)/rear_mount" />
     <origin xyz="${-mount_spacing} 0 0" />
   </joint>
-  <link name="front_mount"></link>
-  <joint name="front_mount_joint" type="fixed">
-    <parent link="mid_mount" />
-    <child link="front_mount" />
+  <link name="$(arg tf_prefix)/front_mount"></link>
+  <joint name="$(arg tf_prefix)/front_mount_joint" type="fixed">
+    <parent link="$(arg tf_prefix)/mid_mount" />
+    <child link="$(arg tf_prefix)/front_mount" />
     <origin xyz="${mount_spacing} 0 0" />
   </joint>
@@ -229,4 +229,4 @@
   <!-- Optional custom includes. -->
   <xacro:include filename="$(optenv JACKAL_URDF_EXTRAS empty.urdf)" />
-  <xacro:include filename="$(find vr_robot_description)/urdf/vr_robot_description.urdf" />
+  <xacro:include filename="$(find vr_robot_description)/urdf/vr_robot_description.urdf.xacro" />
 </robot>

Commit message: Revert "Fix: Add tf_prefix into xacro"
This reverts commit b4f0cb24b7e892a34087f1d696345870020054d3.

File: catkin_ws/src/jackal/jackal_description/urdf/jackal.urdf.xacro (robot description, xacro)
@@ -18,5 +18,5 @@
   <material name="black"><color rgba="0.15 0.15 0.15 1.0" /></material>
   <xacro:macro name="wheel" params="prefix *joint_pose">
-    <link name="$(arg tf_prefix)/${prefix}_wheel_link">
+    <link name="${prefix}_wheel_link">
       <visual>
         <origin xyz="0 0 0" rpy="${PI/2} 0 0"/>
@@ -50,7 +50,7 @@
       <fdir1 value="1 0 0"/>
     </gazebo>
-    <joint name="$(arg tf_prefix)/${prefix}_wheel" type="continuous">
-      <parent link="$(arg tf_prefix)/chassis_link"/>
-      <child link="$(arg tf_prefix)/${prefix}_wheel_link" />
+    <joint name="${prefix}_wheel" type="continuous">
+      <parent link="chassis_link"/>
+      <child link="${prefix}_wheel_link" />
       <xacro:insert_block name="joint_pose" />
       <axis xyz="0 1 0" />
@@ -60,5 +60,5 @@
     <transmission name="${prefix}_wheel_trans">
       <type>transmission_interface/SimpleTransmission</type>
-      <joint name="$(arg tf_prefix)/${prefix}_wheel">
+      <joint name="${prefix}_wheel">
         <hardwareInterface>hardware_interface/VelocityJointInterface</hardwareInterface>
       </joint>
@@ -80,11 +80,11 @@
     <origin xyz="${-wheelbase/2} ${-track/2} ${wheel_vertical_offset}" rpy="0 0 0" />
   </xacro:wheel>
-  <link name="$(arg tf_prefix)/base_link"> </link>
-  <joint name="$(arg tf_prefix)/base_link_joint" type="fixed">
+  <link name="base_link"> </link>
+  <joint name="base_link_joint" type="fixed">
     <origin xyz="0 0 0" rpy="0 0 0" />
-    <parent link="$(arg tf_prefix)/base_link"/>
-    <child link="$(arg tf_prefix)/chassis_link" />
-  </joint>
-  <link name="$(arg tf_prefix)/chassis_link">
+    <parent link="base_link"/>
+    <child link="chassis_link" />
+  </joint>
+  <link name="chassis_link">
     <visual>
       <origin xyz="0 0 ${footprint_vertical_offset}" rpy="${PI/2} 0 ${PI/2}"/>
@@ -112,5 +112,5 @@
   </link>
   <xacro:unless value="$(optenv JACKAL_FRONT_ACCESSORY_FENDER 0)">
-    <link name="$(arg tf_prefix)/front_fender_link">
+    <link name="front_fender_link">
       <visual>
         <geometry>
@@ -122,5 +122,5 @@
   </xacro:unless>
   <xacro:if value="$(optenv JACKAL_FRONT_ACCESSORY_FENDER 0)">
-    <link name="$(arg tf_prefix)/front_fender_link">
+    <link name="front_fender_link">
       <visual>
         <geometry>
@@ -130,18 +130,18 @@
       </visual>
     </link>
-    <link name="$(arg tf_prefix)/front_fender_accessory_link"/>
-    <joint name="$(arg tf_prefix)/front_fender_accessory_joint" type="fixed">
+    <link name="front_fender_accessory_link"/>
+    <joint name="front_fender_accessory_joint" type="fixed">
       <origin xyz="0.25629 0 0.07455" rpy="${PI} 0 0" />
-      <parent link="$(arg tf_prefix)/front_fender_link" />
-      <child link="$(arg tf_prefix)/front_fender_accessory_link" />
+      <parent link="front_fender_link" />
+      <child link="front_fender_accessory_link" />
     </joint>
   </xacro:if>
-  <joint name="$(arg tf_prefix)/front_fender_joint" type="fixed">
+  <joint name="front_fender_joint" type="fixed">
     <origin xyz="0 0 0" rpy="0 0 0"/>
-    <parent link="$(arg tf_prefix)/chassis_link" />
-    <child link="$(arg tf_prefix)/front_fender_link" />
+    <parent link="chassis_link" />
+    <child link="front_fender_link" />
   </joint>
   <xacro:unless value="$(optenv JACKAL_REAR_ACCESSORY_FENDER 0)">
-    <link name="$(arg tf_prefix)/rear_fender_link">
+    <link name="rear_fender_link">
       <visual>
         <geometry>
@@ -153,5 +153,5 @@
   </xacro:unless>
   <xacro:if value="$(optenv JACKAL_REAR_ACCESSORY_FENDER 0)">
-    <link name="$(arg tf_prefix)/rear_fender_link">
+    <link name="rear_fender_link">
       <visual>
         <geometry>
@@ -161,15 +161,15 @@
       </visual>
     </link>
-    <link name="$(arg tf_prefix)/rear_fender_accessory_link"/>
-    <joint name="$(arg tf_prefix)/rear_fender_accessory_joint" type="fixed">
+    <link name="rear_fender_accessory_link"/>
+    <joint name="rear_fender_accessory_joint" type="fixed">
       <origin xyz="0.25629 0 0.07455" rpy="${PI} 0 0" />
-      <parent link="$(arg tf_prefix)/rear_fender_link" />
-      <child link="$(arg tf_prefix)/rear_fender_accessory_link" />
+      <parent link="rear_fender_link" />
+      <child link="rear_fender_accessory_link" />
     </joint>
   </xacro:if>
-  <joint name="$(arg tf_prefix)/rear_fender_joint" type="fixed">
+  <joint name="rear_fender_joint" type="fixed">
     <origin xyz="0 0 0" rpy="0 0 ${PI}"/>
-    <parent link="$(arg tf_prefix)/chassis_link" />
-    <child link="$(arg tf_prefix)/rear_fender_link" />
+    <parent link="chassis_link" />
+    <child link="rear_fender_link" />
   </joint>
   <!-- TODO: Make this internal_imu_link or something, and use a mixed-in xacro
@@ -177,5 +177,5 @@
        always points to the "active" IMU. When an upgrade IMU is connected, the
        internal_imu_link should remain, but imu_link should point to the upgrade one. -->
-  <link name="$(arg tf_prefix)/imu_link">
+  <link name="imu_link">
     <inertial>
       <mass value="0.001"/>
@@ -184,10 +184,10 @@
     </inertial>
   </link>
-  <joint name="$(arg tf_prefix)/imu_joint" type="fixed">
-    <parent link="$(arg tf_prefix)/chassis_link" />
-    <child link="$(arg tf_prefix)/imu_link" />
+  <joint name="imu_joint" type="fixed">
+    <parent link="chassis_link" />
+    <child link="imu_link" />
   </joint>
   <!-- TODO: Same note as applies to imu_link -->
-  <link name="$(arg tf_prefix)/navsat_link">
+  <link name="navsat_link">
     <visual>
       <geometry>
@@ -198,25 +198,25 @@
     </visual>
   </link>
-  <joint name="$(arg tf_prefix)/navsat_joint" type="fixed">
-    <parent link="$(arg tf_prefix)/chassis_link" />
-    <child link="$(arg tf_prefix)/navsat_link" />
+  <joint name="navsat_joint" type="fixed">
+    <parent link="chassis_link" />
+    <child link="navsat_link" />
     <origin xyz="-0.180 0.126 0.1815" />
   </joint>
-  <link name="$(arg tf_prefix)/mid_mount"></link>
-  <joint name="$(arg tf_prefix)/mid_mount_joint" type="fixed">
-    <parent link="$(arg tf_prefix)/chassis_link" />
-    <child link="$(arg tf_prefix)/mid_mount" />
+  <link name="mid_mount"></link>
+  <joint name="mid_mount_joint" type="fixed">
+    <parent link="chassis_link" />
+    <child link="mid_mount" />
     <origin xyz="0 0 ${chassis_height}" />
   </joint>
-  <link name="$(arg tf_prefix)/rear_mount"></link>
-  <joint name="$(arg tf_prefix)/rear_mount_joint" type="fixed">
-    <parent link="$(arg tf_prefix)/mid_mount" />
-    <child link="$(arg tf_prefix)/rear_mount" />
+  <link name="rear_mount"></link>
+  <joint name="rear_mount_joint" type="fixed">
+    <parent link="mid_mount" />
+    <child link="rear_mount" />
     <origin xyz="${-mount_spacing} 0 0" />
   </joint>
-  <link name="$(arg tf_prefix)/front_mount"></link>
-  <joint name="$(arg tf_prefix)/front_mount_joint" type="fixed">
-    <parent link="$(arg tf_prefix)/mid_mount" />
-    <child link="$(arg tf_prefix)/front_mount" />
+  <link name="front_mount"></link>
+  <joint name="front_mount_joint" type="fixed">
+    <parent link="mid_mount" />
+    <child link="front_mount" />
     <origin xyz="${mount_spacing} 0 0" />
   </joint>
@@ -229,4 +229,4 @@
   <!-- Optional custom includes. -->
   <xacro:include filename="$(optenv JACKAL_URDF_EXTRAS empty.urdf)" />
-  <xacro:include filename="$(find vr_robot_description)/urdf/vr_robot_description.urdf.xacro" />
+  <xacro:include filename="$(find vr_robot_description)/urdf/vr_robot_description.urdf" />
 </robot>
