Commit message: Feat: Add scan filter

File: catkin_ws/src/jackal/jackal_nctu_description/urdf/jackal_nctu_description.urdf (robot description, URDF)
Before this commit: robot jackal_nctu_description, 13 links, 13 joints
Joints:
- joint velodyne_joint: origin xyz=0.12 0 0.485304161264951 rpy=0 0 0 -> xyz=0.17 0 0.6 rpy=0 0 0
