Commit message: FIx: Remove velodyne2 camera robot descriptions

File: catkin_ws/src/jackal/guiding_robot_description/urdf/guiding_robot_description.urdf (robot description, URDF)
Before this commit: robot guiding_robot_description, 14 links, 14 joints
Links:
- removed link camera_link
- removed link camera_pan_link
- removed link camera_tilt_link
- removed link velodyne2
- removed link velodyne2_layer_link
Joints:
- removed joint camera_joint
- removed joint camera_pan_joint
- removed joint camera_tilt_joint
- removed joint velodyne2_joint
- removed joint velodyne2_layer_joint

Commit message: FIx: Remove mmwave in robot descriptions

File: catkin_ws/src/jackal/guiding_robot_description/urdf/guiding_robot_description.urdf (robot description, URDF)
Before this commit: robot guiding_robot_description, 9 links, 9 joints
Links:
- removed link camera_layer_link
- removed link guiding_base_link
- removed link mmwave_layer_link
- removed link mmwave_left_back_link
- removed link mmwave_left_front_link
- removed link mmwave_right_back_link
- removed link mmwave_right_front_link
- removed link velodyne1
- removed link velodyne_layer_link
- added link velodyne, mass 0.639680330048926; collision mesh filename=package://guiding_robot_description/meshes/velodyne_link.STL; visual mesh filename=package://guiding_robot_description/meshes/velodyne_link.STL
Joints:
- removed joint camera_layer_joint
- removed joint guiding_base_joint
- removed joint mmwave_layer_joint
- removed joint mmwave_left_back_joint
- removed joint mmwave_left_front_joint
- removed joint mmwave_right_back_joint
- removed joint mmwave_right_front_joint
- removed joint velodyne_layer_joint
- joint velodyne_joint: child velodyne1 -> velodyne; parent velodyne_layer_link -> base_link
