Commit message: Feat: Update jackal vr-robot-description

File: catkin_ws/src/jackal/vr_robot_description/urdf/vr_robot_description.urdf (robot description, URDF)
Before this commit: robot guiding_robot_description, 1 links, 1 joints
Links:
- link velodyne: geometry collision mesh filename=package://vr_robot_description/meshes/velodyne_link.STL; visual mesh filename=package://vr_robot_description/meshes/velodyne_link.STL
Joints:
- joint velodyne_joint: origin xyz=0 0 0.0383041612649508 rpy=0 0 0 -> xyz=0.17 0 0.45 rpy=0 0 0

Commit message: Feat: Add axis camera link

File: catkin_ws/src/jackal/vr_robot_description/urdf/vr_robot_description.urdf (robot description, URDF)
Before this commit: robot vr_robot_description, 1 links, 1 joints
Joints:
- added joint axis_camera_joint: type fixed, parent base_link, child axis_camera_link, origin xyz=0.017 0 0 rpy=-1.5 0 0, axis 0 0 0

Commit message: Fix: axis camera link not found

File: catkin_ws/src/jackal/vr_robot_description/urdf/vr_robot_description.urdf (robot description, URDF)
Before this commit: robot vr_robot_description, 1 links, 2 joints
Links:
- added link axis_camera_link, mass 0.0460103793451425; collision mesh filename=package://guiding_robot_description/meshes/camera_pan_link.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; visual mesh filename=package://guiding_robot_description/meshes/camera_pan_link.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

Commit message: Fix: robot description pkg rename

File: catkin_ws/src/jackal/vr_robot_description/urdf/vr_robot_description.urdf (robot description, URDF)
Before this commit: robot vr_robot_description, 2 links, 2 joints
Links:
- link axis_camera_link: geometry collision mesh filename=package://vr_robot_description/meshes/camera_pan_link.STL; visual mesh filename=package://vr_robot_description/meshes/camera_pan_link.STL
